File: pcb/pcbRadon.sch (KiCad schematic (older format))
At the start: 13 parts

Commit message: Add Kicad PCB files
Parts:
- removed U?: AP131-15, TO_SOT_Packages_SMD:SOT-23-5, symbol AP131-15
- added U2: Step-down, radon:Step-Down, symbol Step-down
- J1: renamed from J?; footprint (none) -> Pin_Headers:Pin_Header_Straight_1x02_Pitch2.54mm
- J2: renamed from J?; footprint (none) -> Connectors:BARREL_JACK
- J3: renamed from J?; footprint (none) -> Pin_Headers:Pin_Header_Straight_1x06_Pitch2.54mm
- J4: renamed from J?; footprint (none) -> Pin_Headers:Pin_Header_Straight_1x04_Pitch2.54mm
- JP1, JP2: renamed from JP?; footprint (none) -> Pin_Headers:Pin_Header_Straight_1x02_Pitch2.54mm
- R1, R2, R3: renamed from R?; footprint (none) -> Resistors_THT:R_Axial_DIN0207_L6.3mm_D2.5mm_P7.62mm_Horizontal
- U1: renamed from U?; footprint (none) -> radon:WEMOS_D1_TH
- gave numbers to parts that had none: 2
Connections:
- net GND: now also U2.4 (IN-)
- net VCC: now also U2.1 (OUT+)
- net VDD: now also U2.3 (IN+)
- no-connect marks 2 -> 6
